File: air-machine-motherboard/button-line.kicad_sch (KiCad schematic)
At the start: 16 parts, among them J2 B1, J5 B3, J7 B2, J8 B4

Commit message: wireles air machine motherboard
Changed lines of the file:
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@@
 (kicad_sch (version 20230121) (generator eeschema)
   (paper "A4")
-  (junction (at 132.08 78.74) (diameter 0) (color 0 0 0 0)
+  (junction (at 191.77 78.74) (diameter 0) (color 0 0 0 0)
   )
   (junction (at 255.27 77.47) (diameter 0) (color 0 0 0 0)
@@
   (junction (at 109.22 78.74) (diameter 0) (color 0 0 0 0)
   )
-  (junction (at 191.77 78.74) (diameter 0) (color 0 0 0 0)
+  (junction (at 132.08 78.74) (diameter 0) (color 0 0 0 0)
   )
   (junction (at 73.66 78.74) (diameter 0) (color 0 0 0 0)
@@
     (stroke (width 0) (type default))
   )
+  (wire (pts (xy 255.27 77.47) (xy 262.89 77.47))
+    (stroke (width 0) (type default))
+  )
   (wire (pts (xy 168.91 88.9) (xy 168.91 92.71))
     (stroke (width 0) (type default))
@@
     (stroke (width 0) (type default))
   )
-  (wire (pts (xy 255.27 77.47) (xy 267.97 77.47))
-    (stroke (width 0) (type default))
-  )
-  (wire (pts (xy 73.66 78.74) (xy 86.36 78.74))
-    (stroke (width 0) (type default))
-  )
   (wire (pts (xy 66.04 78.74) (xy 73.66 78.74))
     (stroke (width 0) (type default))
   )
   (wire (pts (xy 220.98 80.01) (xy 220.98 91.44))
+    (stroke (width 0) (type default))
+  )
+  (wire (pts (xy 73.66 78.74) (xy 81.28 78.74))
+    (stroke (width 0) (type default))
+  )
+  (wire (pts (xy 132.08 78.74) (xy 138.43 78.74))
     (stroke (width 0) (type default))
   )
@@
     (stroke (width 0) (type default))
   )
-  (wire (pts (xy 191.77 78.74) (xy 204.47 78.74))
-    (stroke (width 0) (type default))
-  )
   (wire (pts (xy 39.37 78.74) (xy 50.8 78.74))
     (stroke (width 0) (type default))
@@
     (stroke (width 0) (type default))
   )
-  (wire (pts (xy 132.08 78.74) (xy 144.78 78.74))
+  (wire (pts (xy 191.77 78.74) (xy 199.39 78.74))
     (stroke (width 0) (type default))
   )
@@
     (stroke (width 0) (type default))
   )
-  (label "OK" (at 204.47 78.74 180) (fields_autoplaced)
-    (effects (font (size 1.27 1.27)) (justify right bottom))
+  (global_label "OK" (shape input) (at 199.39 78.74 0) (fields_autoplaced)
+    (effects (font (size 1.27 1.27)) (justify left))
+    (property "Intersheetrefs" "${INTERSHEET_REFS}" (at 204.8963 78.74 0)
+      (effects (font (size 1.27 1.27)) (justify left) hide)
+    )
   )
-  (label "DEC" (at 144.78 78.74 180) (fields_autoplaced)
-    (effects (font (size 1.27 1.27)) (justify right bottom))
+  (global_label "INC" (shape input) (at 81.28 78.74 0) (fields_autoplaced)
+    (effects (font (size 1.27 1.27)) (justify left))
+    (property "Intersheetrefs" "${INTERSHEET_REFS}" (at 87.3911 78.74 0)
+      (effects (font (size 1.27 1.27)) (justify left) hide)
+    )
   )
-  (label "INC" (at 86.36 78.74 180) (fields_autoplaced)
-    (effects (font (size 1.27 1.27)) (justify right bottom))
+  (global_label "DEC" (shape input) (at 138.43 78.74 0) (fields_autoplaced)
+    (effects (font (size 1.27 1.27)) (justify left))
+    (property "Intersheetrefs" "${INTERSHEET_REFS}" (at 145.0248 78.74 0)
+      (effects (font (size 1.27 1.27)) (justify left) hide)
+    )
   )
-  (label "EMC" (at 267.97 77.47 180) (fields_autoplaced)
-    (effects (font (size 1.27 1.27)) (justify right bottom))
+  (global_label "EMC" (shape input) (at 262.89 77.47 0) (fields_autoplaced)
+    (effects (font (size 1.27 1.27)) (justify left))
+    (property "Intersheetrefs" "${INTERSHEET_REFS}" (at 269.6662 77.47 0)
+      (effects (font (size 1.27 1.27)) (justify left) hide)
+    )
   )
   (symbol (lib_id "power:GND") (at 157.48 92.71 0) (unit 1)
