File: air-machine-motherboard/mcu-line.kicad_sch (KiCad schematic)
At the start: 8 parts, among them J4 CODE, U1 ESP32-WROOM-32D

Commit message: wireles air machine motherboard
Connections:
- net DEC: no longer names the net of U1.9 (IO33)
- net EMC: no longer names the net of U1.7 (IO35)
- net INC: no longer names the net of U1.8 (IO32)
- net OK: no longer names the net of U1.6 (IO34)
Changed lines of the file:
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@@
   (no_connect (at 102.87 109.22))
   (no_connect (at 133.35 78.74))
-  (wire (pts (xy 133.35 127) (xy 139.7 127))
-    (stroke (width 0) (type default))
-  )
   (wire (pts (xy 85.09 63.5) (xy 85.09 66.04))
     (stroke (width 0) (type default))
@@
   )
   (wire (pts (xy 71.12 54.61) (xy 71.12 55.88))
+    (stroke (width 0) (type default))
+  )
+  (wire (pts (xy 133.35 109.22) (xy 147.32 109.22))
     (stroke (width 0) (type default))
   )
@@
     (stroke (width 0) (type default))
   )
+  (wire (pts (xy 133.35 111.76) (xy 147.32 111.76))
+    (stroke (width 0) (type default))
+  )
   (wire (pts (xy 97.79 54.61) (xy 97.79 57.15))
     (stroke (width 0) (type default))
@@
     (stroke (width 0) (type default))
   )
-  (wire (pts (xy 133.35 111.76) (xy 153.67 111.76))
-    (stroke (width 0) (type default))
-  )
   (wire (pts (xy 187.96 73.66) (xy 187.96 74.93))
-    (stroke (width 0) (type default))
-  )
-  (wire (pts (xy 133.35 124.46) (xy 139.7 124.46))
-    (stroke (width 0) (type default))
-  )
-  (wire (pts (xy 133.35 109.22) (xy 142.24 109.22))
-    (stroke (width 0) (type default))
-  )
-  (wire (pts (xy 133.35 121.92) (xy 139.7 121.92))
     (stroke (width 0) (type default))
   )
@@
     (stroke (width 0) (type default))
   )
-  (wire (pts (xy 133.35 96.52) (xy 138.43 96.52))
+  (wire (pts (xy 133.35 96.52) (xy 147.32 96.52))
     (stroke (width 0) (type default))
   )
@@
     (stroke (width 0) (type default))
   )
-  (wire (pts (xy 133.35 119.38) (xy 139.7 119.38))
-    (stroke (width 0) (type default))
-  )
   (wire (pts (xy 203.2 74.93) (xy 203.2 76.2))
     (stroke (width 0) (type default))
@@
     (effects (font (size 1.27 1.27)) (justify left bottom))
   )
-  (label "MOTOR-SG" (at 153.67 111.76 180) (fields_autoplaced)
-    (effects (font (size 1.27 1.27)) (justify right bottom))
-  )
-  (label "LED" (at 142.24 109.22 180) (fields_autoplaced)
-    (effects (font (size 1.27 1.27)) (justify right bottom))
-  )
-  (label "INC" (at 139.7 119.38 180) (fields_autoplaced)
-    (effects (font (size 1.27 1.27)) (justify right bottom))
-  )
-  (label "EMC" (at 139.7 127 180) (fields_autoplaced)
-    (effects (font (size 1.27 1.27)) (justify right bottom))
-  )
-  (label "DEC" (at 139.7 121.92 180) (fields_autoplaced)
-    (effects (font (size 1.27 1.27)) (justify right bottom))
-  )
   (label "IO0" (at 148.59 68.58 180) (fields_autoplaced)
     (effects (font (size 1.27 1.27)) (justify right bottom))
   )
   (label "TX" (at 148.59 71.12 180) (fields_autoplaced)
-    (effects (font (size 1.27 1.27)) (justify right bottom))
-  )
-  (label "OK" (at 139.7 124.46 180) (fields_autoplaced)
     (effects (font (size 1.27 1.27)) (justify right bottom))
   )
@@
     (effects (font (size 1.27 1.27)) (justify right bottom))
   )
+  (global_label "LED" (shape input) (at 147.32 109.22 0) (fields_autoplaced)
+    (effects (font (size 1.27 1.27)) (justify left))
+    (property "Intersheetrefs" "${INTERSHEET_REFS}" (at 153.6729 109.22 0)
+      (effects (font (size 1.27 1.27)) (justify left) hide)
+    )
+  )
+  (global_label "MOTOR-SG" (shape input) (at 147.32 111.76 0) (fields_autoplaced)
+    (effects (font (size 1.27 1.27)) (justify left))
+    (property "Intersheetrefs" "${INTERSHEET_REFS}" (at 160.6277 111.76 0)
+      (effects (font (size 1.27 1.27)) (justify left) hide)
+    )
+  )
   (global_label "SDA" (shape input) (at 147.32 104.14 0) (fields_autoplaced)
     (effects (font (size 1.27 1.27)) (justify left))
@@
     )
   )
-  (global_label "G" (shape input) (at 138.43 96.52 0) (fields_autoplaced)
+  (global_label "G" (shape input) (at 147.32 96.52 0) (fields_autoplaced)
     (effects (font (size 1.27 1.27)) (justify left))
-    (property "Intersheetrefs" "${INTERSHEET_REFS}" (at 142.6852 96.52 0)
+    (property "Intersheetrefs" "${INTERSHEET_REFS}" (at 151.5752 96.52 0)
       (effects (font (size 1.27 1.27)) (justify left) hide)
     )
