File: air-machine-motherboard/output-line.kicad_sch (KiCad schematic)
At the start: 11 parts, among them J10 MOTOR, J9 LED, Q2 IRF540N, Q4 2N7002, Q5 2N7002

Commit message: wireles air machine motherboard
Changed lines of the file:
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@@
     (stroke (width 0) (type default))
   )
-  (label "LED" (at 97.79 73.66 0) (fields_autoplaced)
-    (effects (font (size 1.27 1.27)) (justify left bottom))
+  (global_label "MOTOR-SG" (shape input) (at 194.31 81.28 180) (fields_autoplaced)
+    (effects (font (size 1.27 1.27)) (justify right))
+    (property "Intersheetrefs" "${INTERSHEET_REFS}" (at 181.0023 81.28 0)
+      (effects (font (size 1.27 1.27)) (justify right) hide)
+    )
   )
-  (label "MOTOR-SG" (at 194.31 81.28 0) (fields_autoplaced)
-    (effects (font (size 1.27 1.27)) (justify left bottom))
+  (global_label "LED" (shape input) (at 97.79 73.66 180) (fields_autoplaced)
+    (effects (font (size 1.27 1.27)) (justify right))
+    (property "Intersheetrefs" "${INTERSHEET_REFS}" (at 91.4371 73.66 0)
+      (effects (font (size 1.27 1.27)) (justify right) hide)
+    )
   )
   (symbol (lib_id "power:+3.3V") (at 208.28 66.04 0) (unit 1)
