File: air-machine-motherboard/piezzo.kicad_pcb (KiCad board)
At the start: 2 copper layers, 0 parts

Commit message: wireles air machine motherboard
Parts:
- added C1: 1uF, Capacitor_SMD:C_0603_1608Metric, F.Cu at (53.2, 18.4)
- added C10: 10uF, Capacitor_SMD:C_0603_1608Metric, F.Cu at (13.2, 23.6)
- added C11: 4.7uF, Capacitor_SMD:C_0603_1608Metric, F.Cu at (25.3, 31.4)
- added C12: 10uF, Capacitor_SMD:C_0603_1608Metric, F.Cu at (12.9, 37.1)
- added C13: 4.7uF, Capacitor_SMD:C_0603_1608Metric, F.Cu at (25.6, 43.2)
- added C2: 47uH, Capacitor_SMD:C_0603_1608Metric, F.Cu at (54.8, 21.5)
- added C3: 47uH, Capacitor_THT:CP_Radial_D5.0mm_P2.50mm, F.Cu at (17.6, 6.10)
- added C4: 10uF, Capacitor_SMD:C_0603_1608Metric, F.Cu at (68.8, 38.0)
- added C5: 1uF, Capacitor_SMD:C_0603_1608Metric, F.Cu at (68.8, 41.2)
- added C6: 100nF, Capacitor_SMD:C_0603_1608Metric, F.Cu at (42.2, 74.2)
- added C7: 100nF, Capacitor_SMD:C_0603_1608Metric, F.Cu at (22.7, 72.0)
- added C8: 330nF, Capacitor_SMD:C_0603_1608Metric, F.Cu at (23.9, 3.60)
- added C9: 330nF, Capacitor_SMD:C_0603_1608Metric, F.Cu at (17.3, 14.2)
- added D1: SMBJ30CA, Diode_SMD:D_MELF, F.Cu at (28.0, 5.98)
- added D10: RS1M, Diode_SMD:D_MELF, F.Cu at (7.86, 24.3)
- added D11: RS1M, Diode_SMD:D_MELF, F.Cu at (7.89, 37.8)
- added D12: RS1A, Diode_SMD:D_MELF, F.Cu at (76.9, 15.7)
- added D13: RS1A, Diode_SMD:D_MELF, F.Cu at (7.92, 67.5)
- added D14: RS1A, Diode_SMD:D_MELF, F.Cu at (63.9, 5.78)
- added D2: SMAJ10CA, Diode_SMD:D_MELF, F.Cu at (52.1, 70.6)
- added D4: SMAJ10CA, Diode_SMD:D_MELF, F.Cu at (64.6, 68.6)
- added D6: SMAJ10CA, Diode_SMD:D_MELF, F.Cu at (21.1, 67.0)
- added D9: SMBJ30CA, Diode_SMD:D_MELF, F.Cu at (11.4, 17.1)
- added J10: MOTOR, Connector_PinHeader_2.54mm:PinHeader_1x02_P2.54mm_Vertical, F.Cu at (2.75, 67.3)
- added J2: OUT, Connector_PinHeader_2.54mm:PinHeader_1x02_P2.54mm_Vertical, F.Cu at (6.42, 6.14)
- added J3: OUT, Connector_PinHeader_2.54mm:PinHeader_1x02_P2.54mm_Vertical, F.Cu at (48.7, 15.8)
- added J4: CODE, Connector_PinSocket_2.54mm:PinSocket_2x04_P2.54mm_Vertical, F.Cu at (46.7, 74.9)
- added J6: LCD, Connector_PinHeader_2.54mm:PinHeader_1x04_P2.54mm_Vertical, F.Cu at (23.5, 76.2)
- added J9: LED, Connector_PinHeader_2.54mm:PinHeader_1x02_P2.54mm_Vertical, F.Cu at (3.02, 52.8)
- added L1: 220uH, Inductor_THT:L_Radial_D10.0mm_P5.00mm_Fastron_07M, F.Cu at (62.1, 21.5)
- added Q1: BU407, Package_TO_SOT_THT:TO-220-3_Vertical, F.Cu at (68.4, 13.2)
- added Q2: 2N7002, Package_TO_SOT_SMD:SOT-23, F.Cu at (8.55, 59.6)
- added Q3: IRF9540N, Package_TO_SOT_THT:TO-220-3_Vertical, F.Cu at (56.9, 3.07)
- added Q4: IRF540N, Package_TO_SOT_THT:TO-220-3_Vertical, F.Cu at (13.2, 49.9)
- added Q5: 2N7002, Package_TO_SOT_SMD:SOT-23, F.Cu at (8.81, 73.7)
- added R1: 2.2K, Resistor_SMD:R_0603_1608Metric, F.Cu at (56.9, 13.2)
- added R12: 47K, Resistor_SMD:R_0603_1608Metric, F.Cu at (52.3, 3.98)
- added R13: 47K, Resistor_SMD:R_0603_1608Metric, F.Cu at (15.2, 61.4)
- added R14: 4.7K, Resistor_SMD:R_0603_1608Metric, F.Cu at (4.24, 58.8)
- added R15: 1K, Resistor_SMD:R_0603_1608Metric, F.Cu at (13.1, 56.8)
- added R16: 47K, Resistor_SMD:R_0603_1608Metric, F.Cu at (9.00, 56.0)
- added R17: 47K, Resistor_SMD:R_0603_1608Metric, F.Cu at (14.1, 73.9)
- added R2: 2.2K, Resistor_SMD:R_0603_1608Metric, F.Cu at (56.8, 16.6)
- added R3: 10K, Resistor_SMD:R_0603_1608Metric, F.Cu at (68.8, 44.2)
- added U1: ESP32-WROOM-32D, RF_Module:ESP32-WROOM-32D, F.Cu at (62.6, 56.5)
- added U2: LM7812_TO220, Package_TO_SOT_THT:TO-220-3_Vertical, F.Cu at (27.6, 13.3)
- added U3: AMS1117-3.3, Package_TO_SOT_SMD:SOT-223-3_TabPin2, F.Cu at (19.1, 27.4)
- added U4: AMS1117-3.3, Package_TO_SOT_SMD:SOT-223-3_TabPin2, F.Cu at (19.1, 40.8)
Routing:
- net +24V: track 0.00 -> 162.6 mm
- net +3.3V: track 68.1 -> 197.6 mm, vias 0 -> 2
- net G: track 124.3 -> 4.63 mm
- net GND: track 107.4 -> 0.00 mm
- net MOTOR-SG: track 0.00 -> 73.3 mm, vias 0 -> 2
- net LED: track 0.00 -> 65.4 mm, vias 0 -> 2
- net SCL: track 0.00 -> 56.6 mm, vias 0 -> 1
- net SDA: track 0.00 -> 49.0 mm, vias 0 -> 1
- net +12V: track 0.00 -> 39.3 mm
- net Net-(D12-K): track 0.00 -> 36.7 mm
- net /mcu-line/RX: track 0.00 -> 28.6 mm
- net Net-(D12-A): track 0.00 -> 23.9 mm
- net /mcu-line/TX: track 0.00 -> 21.1 mm
- net /IO0: track 21.0 -> 0.00 mm
- net Net-(Q1-B): track 0.00 -> 13.4 mm
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- added copper zone on B.Cu, net GND
- added copper zone on F.Cu, net GND
Other:
- board outline added: 80 x 80 mm
