File: air-machine-motherboard/piezzo.kicad_sch (KiCad schematic)
At the start: 0 parts

Commit message: wireles air machine motherboard
Other:
- removed sheet button-line
Changed lines of the file:
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@@
-    )
-  )
-  (sheet (at 165.1 20.32) (size 38.1 16.51) (fields_autoplaced)
-    (stroke (width 0.1524) (type solid))
-    (fill (color 0 0 0 0.0000))
-    (property "Sheetname" "button-line" (at 165.1 19.6084 0)
-      (effects (font (size 1.27 1.27)) (justify left bottom))
-    )
-    (property "Sheetfile" "button-line.kicad_sch" (at 165.1 37.4146 0)
-      (effects (font (size 1.27 1.27)) (justify left top))
-    )
-    (instances
-      (project "piezzo"
-        (path "/2a569c31-bb52-4c3d-ae7f-45f2860154f7" (page "6"))
-      )
     )
   )
