File: air-machine-motherboard/power.kicad_sch (KiCad schematic)
At the start: 18 parts, among them J1 MAIN, Q3 IRF9540N, U2 LM7812_TO220, U3 AMS1117-3.3, U4 AMS1117-3.3

Commit message: wireles air machine motherboard
Parts:
- removed D14: SMBJ30CA, Diode_SMD:D_MELF, symbol Device:D_TVS
- removed J1: MAIN, Connector_PinHeader_2.54mm:PinHeader_1x02_P2.54mm_Vertical, symbol Connector_Generic:Conn_01x02
- removed Q3: IRF9540N, Package_TO_SOT_THT:TO-220-3_Vertical, symbol Transistor_FET:IRF9540N
- removed R12: 47K, Resistor_SMD:R_0603_1608Metric, symbol Device:R
- added J3: OUT, Connector_PinHeader_2.54mm:PinHeader_1x02_P2.54mm_Vertical, symbol Connector_Generic:Conn_01x02
Connections:
- net +24V: now also J3.2 (Pin_2)
- net GND: now also J3.1 (Pin_1)
Other:
- note removed: "P KANAL MOSFET İLE PİEZZO HATTI AÇILIP KAPATILIYOR"
